File: hardware/mito.kicad_pcb (KiCad board)
At the start: 2 copper layers, 48 x 32 mm, 31 parts, among them J1 Conn_01x02, J2 Conn_01x07, J3 Conn_01x07, J4 Conn_01x02, J5 Conn_01x05, Q1 MMBT4403, SW1 SW_Push, U1 HX711

Commit message: Upload hardware
Parts:
- removed J2, J3: Conn_01x07, Connector_PinHeader_2.54mm:PinHeader_1x07_P2.54mm_Vertical
- removed J4: Conn_01x02, Connector_Wire:SolderWire-0.1sqmm_1x02_P3.6mm_D0.4mm_OD1mm
- added G***: LOGO, LOGO, B.Cu at (157.0, 102.0)
- added U2: XIAO-ESP32-C3-DIP, xiao:XIAO-nRF52840-SMD, F.Cu at (164.1, 107.2)
- C6, C7: footprint Capacitor_SMD:C_1210_3225Metric -> PCM_JLCPCB:C_0603
- R2: value 8.2K -> 8K2R; footprint Resistor_SMD:R_0603_1608Metric -> PCM_JLCPCB:R_0603
- R3, R4: value 100 -> 100R; footprint Resistor_SMD:R_0603_1608Metric -> PCM_JLCPCB:R_0603
- R5: value 43R -> 150R
- R7, R8: value 10R -> 100R
- moved FRAME1 82.7 mm to (200.1, 176.3)
- moved R5 9.87 mm to (164.0, 95.2), turned to -90 degrees
- moved R7 6.89 mm to (166.5, 95.2), turned to -90 degrees
- moved R8 4.78 mm to (169.0, 95.2), turned to -90 degrees
- moved R6 1.39 mm to (156.0, 95.1)
- moved C7 1.22 mm to (144.4, 95.8)
- moved C3 1.00 mm to (141.4, 95.8)
- moved C6 0.68 mm to (151.0, 95.8)
- moved C4 0.34 mm to (153.0, 101.3)
- moved C5 0.32 mm to (148.0, 95.8)
Connections:
- U1 pad 15: VCC -> unconnected-(U1-RATE-Pad15)
Routing:
- net Net-(SW3-A): track 6.51 -> 25.0 mm, vias 0 -> 1
- net /TARE: track 14.3 -> 3.72 mm
- net Net-(U2-GPIO6/D4/SDA): track 3.52 -> 12.9 mm
- net Net-(D1-RK): track 23.7 -> 15.3 mm
- net Net-(U2-GPIO7/D5/SCL): track 3.52 -> 9.33 mm
- net Net-(D1-GK): track 20.6 -> 16.2 mm
- net /DAT: track 8.80 -> 5.46 mm
- net GND: track 25.2 -> 28.4 mm, vias 8 -> 10
- net /SCK: track 7.31 -> 5.19 mm
- net Net-(U2-GPIO21/D6/TX): track 3.52 -> 4.95 mm
- net /AVDD: track 15.1 -> 16.1 mm
- net Net-(J1-Pin_1): track 17.6 -> 18.5 mm
- net Net-(D1-BK): track 18.6 -> 17.9 mm
- net unconnected-(U2-GPIO8/D8/SCK-Pad9): track 0.00 -> 0.55 mm
- net VCC: track 59.4 -> 59.5 mm, vias 4 -> 3
Other:
- board text removed: "Batt In"
- board text removed: "Batt to Xiao"
- board text removed: "mito"

Commit message: Fix issues with hardware.
Parts:
- removed SW1: SW_Push, Button_Switch_SMD:Panasonic_EVQPUJ_EVQPUA
- added TARE: SW_Push, Button_Switch_SMD:Panasonic_EVQPUJ_EVQPUA, F.Cu at (146.3, 88.0)
- J1: footprint Connector_Wire:SolderWire-0.1sqmm_1x02_P3.6mm_D0.4mm_OD1mm -> Connector_Molex:Molex_PicoBlade_53048-0210_1x02_P1.25mm_Horizontal
- J5: footprint Connector_Wire:SolderWire-0.1sqmm_1x05_P3.6mm_D0.4mm_OD1mm -> Connector_PinHeader_2.54mm:PinHeader_1x05_P2.54mm_Vertical
- R2: value 8K2R -> 8.2K
- R3, R4: value 100R -> 100
- moved R6 5.84 mm to (151.0, 92.1)
- moved J1 5.13 mm to (176.5, 95.7), turned to 0 degrees
- moved J5 1.70 mm to (135.9, 96.6), turned to 0 degrees
- moved G*** 0.98 mm to (156.0, 102.0)
- moved PWR 0.12 mm to (166.0, 88.4)
Connections:
- PWR pad 3: Net-(SW3-A) -> Net-(PWR1-A)
- R6 pad 1: GND -> /TARE
- R6 pad 2: /TARE -> GND
- U2 pad 15: GND -> Net-(PWR1-A)
- U2 pad 16: Net-(SW3-A) -> GND
Routing:
- net Net-(SW3-A): track 25.0 -> 0.00 mm, vias 1 -> 0
- net Net-(PWR1-A): track 0.00 -> 23.1 mm, vias 0 -> 2
- net /TARE: track 3.72 -> 19.7 mm
- net GND: track 28.4 -> 16.9 mm, vias 10 -> 9
- net Net-(J1-Pin_1): track 18.5 -> 16.1 mm
- net /A+: track 8.60 -> 10.0 mm
- net /AVDD: track 16.1 -> 15.3 mm
- net VCC: track 59.5 -> 58.9 mm
Other:
- board text removed: "TARE"
