File: hardware/mito.kicad_pcb (KiCad board)
At the start: 2 copper layers, 48 x 32 mm, 30 parts, among them J1 Conn_01x02, J5 Conn_01x05, Q1 MMBT4403, U1 HX711, U2 XIAO-ESP32-C3-DIP

Commit message: Breakout xiao pins
Parts:
- added J2: Conn_01x04, Connector_PinHeader_2.54mm:PinHeader_1x04_P2.54mm_Vertical, F.Cu at (142.7, 116.0)
Connections:
- U2 pad 1: unconnected-(U2-GPIO2/A0/D0-Pad1) -> Net-(J2-Pin_1)
- U2 pad 2: unconnected-(U2-GPIO3/A1/D1-Pad2) -> Net-(J2-Pin_2)
- U2 pad 3: unconnected-(U2-GPIO4/A2/D2-Pad3) -> Net-(J2-Pin_3)
- U2 pad 4: unconnected-(U2-GPIO5/A3/D3-Pad4) -> Net-(J2-Pin_4)
Routing:
- net Net-(J2-Pin_1): track 0.00 -> 31.0 mm
- net Net-(J2-Pin_4): track 0.00 -> 29.8 mm, vias 0 -> 1
- net Net-(J2-Pin_2): track 0.00 -> 29.5 mm, vias 0 -> 1
- net Net-(J2-Pin_3): track 0.00 -> 28.3 mm
Other:
- board text added: "1"
- board text added: "2"
- board text added: "3"
- board text added: "4"
- board text added: "GPIO"

Commit message: mito V2 pcb
Parts:
- removed PWR: SW_SPDT_321, Button_Switch_THT:SW_Slide_SPDT_Angled_CK_OS102011MA1Q
- removed TARE: SW_Push, Button_Switch_SMD:Panasonic_EVQPUJ_EVQPUA
- added PWR1: SW_SPDT_321, Button_Switch_THT:SW_Slide_SPDT_Angled_CK_OS102011MA1Q, F.Cu at (165.9, 88.5)
- added TARE1: SW_Push, Button_Switch_SMD:Panasonic_EVQPUJ_EVQPUA, F.Cu at (145.9, 88.0)
- J1: footprint Connector_Molex:Molex_PicoBlade_53048-0210_1x02_P1.25mm_Horizontal -> Connector_Wire:SolderWire-0.1sqmm_1x02_P3.6mm_D0.4mm_OD1mm_Relief
- J2: value Conn_01x04 -> Conn_01x06; footprint Connector_PinHeader_2.54mm:PinHeader_1x04_P2.54mm_Vertical -> Connector_PinHeader_2.54mm:PinHeader_1x06_P2.54mm_Vertical
- moved J2 36.4 mm to (178.3, 108.5), turned to 180 degrees
- moved J1 30.7 mm to (151.2, 113.1), turned to -90 degrees
- moved R6 9.58 mm to (141.4, 91.9)
- moved R5 3.20 mm to (167.2, 95.2)
- moved R7 3.20 mm to (169.7, 95.2)
- moved R8 3.20 mm to (172.2, 95.2)
- moved G*** 1.38 mm to (157.0, 103.0)
- moved C1 1.00 mm to (145.8, 112.0)
Connections:
- U1 pad 15: unconnected-(U1-RATE-Pad15) -> VCC
Routing:
- net VCC: track 58.9 -> 84.8 mm
- net Net-(J2-Pin_4): track 29.8 -> 8.92 mm, vias 1 -> 0
- net Net-(J2-Pin_2): track 29.5 -> 8.92 mm, vias 1 -> 0
- net Net-(J2-Pin_3): track 28.3 -> 8.92 mm
- net Net-(J1-Pin_1): track 16.1 -> 33.2 mm
- net Net-(J2-Pin_1): track 31.0 -> 18.3 mm
- net Net-(D1-GK): track 16.2 -> 19.4 mm
- net Net-(D1-RK): track 15.3 -> 18.5 mm
- net Net-(D1-BK): track 17.9 -> 21.1 mm
- net /TARE: track 19.7 -> 21.8 mm
- net Net-(U2-GPIO6/D4/SDA): track 12.9 -> 11.5 mm
- net Net-(U2-GPIO7/D5/SCL): track 9.33 -> 7.96 mm
- net Net-(U2-GPIO21/D6/TX): track 4.95 -> 3.60 mm
- net Net-(PWR1-A): track 23.1 -> 22.2 mm, vias 2 -> 1
Other:
- board text added: "3.3V"
- board text added: "Battery"
- board text added: "D0"
- board text added: "D1"
- board text added: "D2"
- board text added: "D3"
- board text added: "GND"
- board text removed: "1"
- board text removed: "2"
- board text removed: "3"
- board text removed: "4"
- board text removed: "GPIO"
