File: hardware/mito.kicad_sch (KiCad schematic)
At the start: 38 parts, among them J1 Conn_01x02, J2 Conn_01x07, J3 Conn_01x07, J4 Conn_01x02, J5 Conn_01x05, Q1 MMBT4403, SW1 SW_Push, SW3 SW_SPDT_321, U1 HX711

Commit message: Upload hardware
Parts:
- removed J2, J3: Conn_01x07, Connector_PinHeader_2.54mm:PinHeader_1x07_P2.54mm_Vertical, symbol Connector_Generic:Conn_01x07
- removed J4: Conn_01x02, Connector_Wire:SolderWire-0.1sqmm_1x02_P3.6mm_D0.4mm_OD1mm, symbol Connector_Generic:Conn_01x02
- added U2: XIAO-ESP32-C3-DIP, xiao:XIAO-nRF52840-SMD, symbol xiao:XIAO-ESP32-C3-DIP
- C6, C7: footprint Capacitor_SMD:C_1210_3225Metric -> PCM_JLCPCB:C_0603
- R5: value 180R -> 150R
Connections:
- net DAT: now also U2.10 (GPIO9/D9/MISO)
- net GND: now also U2.13 (GND), U2.15 (Bat-)
- net SCK: now also U2.11 (GPIO10/D10/MOSI)
- net TARE: now also U2.8 (GPIO20/D7/RX)
- net VCC: now also U2.12 (VCC_3V3); no longer U1.15 (RATE)
- net at SW3.3 (A): now also U2.16 (Bat+)
- net at R7.2: now also U2.6 (GPIO7/D5/SCL)
- net at R8.2: now also U2.7 (GPIO21/D6/TX)
- net at R5.2: now also U2.5 (GPIO6/D4/SDA)
Other:
- note added: "= 3.08V"
- note removed: "Battery to XIAO"
- note removed: "XIAO Headers"
- moved on the sheet: J1, R6, SW1, SW3

Commit message: Fix issues with hardware.
Parts:
- J1: footprint Connector_Wire:SolderWire-0.1sqmm_1x02_P3.6mm_D0.4mm_OD1mm -> Connector_Molex:Molex_PicoBlade_53048-0210_1x02_P1.25mm_Horizontal
- J5: footprint Connector_Wire:SolderWire-0.1sqmm_1x05_P3.6mm_D0.4mm_OD1mm -> Connector_PinHeader_2.54mm:PinHeader_1x05_P2.54mm_Vertical
- renumbered SW3 to PWR1, SW1 to TARE1
Connections:
- net GND: now also R6.2, U2.16 (Bat-); no longer R6.1, TARE1.1, U2.15 (Bat-)
- net TARE: now also R6.1, TARE1.1; no longer R6.2
- net at PWR1.3 (A): now also U2.15 (Bat+); no longer U2.16 (Bat+)
Other:
- moved on the sheet: R6
Changed lines of the file:
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@@
-	(wire
-		(pts
-			(xy 233.68 125.73) (xy 248.92 125.73)
-		)
-		(stroke
-			(width 0)
-			(type default)
-		)
-	)
 	(wire
 		(pts
@@
 	(wire
 		(pts
+			(xy 233.68 110.49) (xy 233.68 123.19)
+		)
+		(stroke
+			(width 0)
+			(type default)
+		)
+	)
+	(wire
+		(pts
 			(xy 101.6 152.4) (xy 109.22 152.4)
 		)
@@
 	(wire
 		(pts
-			(xy 229.87 123.19) (xy 241.3 123.19)
-		)
-		(stroke
-			(width 0)
-			(type default)
-		)
-	)
-	(wire
-		(pts
 			(xy 82.55 81.28) (xy 82.55 88.9)
 		)
@@
 		)
 	)
-	(wire
-		(pts
-			(xy 217.17 77.47) (xy 217.17 82.55)
-		)
-		(stroke
-			(width 0)
-			(type default)
-		)
-	)
 	(polyline
 		(pts
@@
 	(wire
 		(pts
+			(xy 229.87 125.73) (xy 248.92 125.73)
+		)
+		(stroke
+			(width 0)
+			(type default)
+		)
+	)
+	(wire
+		(pts
 			(xy 269.24 72.39) (xy 269.24 90.17)
 		)
@@
 	(wire
 		(pts
+			(xy 219.71 66.04) (xy 217.17 66.04)
+		)
+		(stroke
+			(width 0)
+			(type default)
+		)
+	)
+	(wire
+		(pts
 			(xy 144.78 129.54) (xy 144.78 132.08)
 		)
@@
 	(wire
 		(pts
-			(xy 217.17 69.85) (xy 217.17 66.04)
+			(xy 217.17 66.04) (xy 217.17 82.55)
 		)
 		(stroke
@@
 	(wire
 		(pts
-			(xy 233.68 125.73) (xy 233.68 110.49)
-		)
-		(stroke
-			(width 0)
-			(type default)
-		)
-	)
-	(wire
-		(pts
 			(xy 111.76 63.5) (xy 111.76 60.96)
 		)
@@
 	(wire
 		(pts
-			(xy 229.87 123.19) (xy 229.87 110.49)
-		)
-		(stroke
-			(width 0)
-			(type default)
-		)
-	)
-	(wire
-		(pts
 			(xy 270.51 68.58) (xy 274.32 68.58)
 		)
@@
 	(wire
 		(pts
+			(xy 241.3 123.19) (xy 233.68 123.19)
+		)
+		(stroke
+			(width 0)
+			(type default)
+		)
+	)
+	(wire
+		(pts
 			(xy 209.55 93.98) (xy 219.71 93.98)
 		)
@@
 			(width 0.1524)
 			(type solid)
+		)
+	)
+	(wire
+		(pts
+			(xy 229.87 125.73) (xy 229.87 110.49)
+		)
+		(stroke
+			(width 0)
+			(type default)
 		)
 	)
@@
 		(dnp no)
 		(fields_autoplaced yes)
-		(property "Reference" "SW3"
+		(property "Reference" "PWR1"
 			(at 246.38 111.76 0)
 			(effects
@@
 			(project "mito"
 				(path "/7828b8a8-8a30-49cd-9e74-a278024fdbdb"
-					(reference "SW3")
+					(reference "PWR1")
 					(unit 1)
 				)
@@
 	(symbol
 		(lib_id "SparkFun_HX711_Load_Cell-eagle-import:GND")
-		(at 219.71 66.04 90)
+		(at 229.87 66.04 90)
 		(unit 1)
 		(exclude_from_sim no)
@@
 		(dnp no)
 		(property "Reference" "#GND07"
-			(at 219.71 66.04 0)
+			(at 229.87 66.04 0)
 			(effects
 				(font
@@
 		)
 		(property "Value" "GND"
-			(at 222.25 68.58 0)
+			(at 232.41 68.58 0)
 			(effects
 				(font
@@
 		)
 		(property "Footprint" ""
-			(at 219.71 66.04 0)
+			(at 229.87 66.04 0)
 			(effects
 				(font
@@
 		)
 		(property "Datasheet" ""
-			(at 219.71 66.04 0)
+			(at 229.87 66.04 0)
 			(effects
 				(font
@@
 		)
 		(property "Description" ""
-			(at 219.71 66.04 0)
+			(at 229.87 66.04 0)
 			(effects
 				(font
@@
 		(dnp no)
 		(fields_autoplaced yes)
-		(property "Reference" "SW1"
+		(property "Reference" "TARE1"
 			(at 212.09 66.04 0)
 			(effects
@@
 			(project ""
 				(path "/7828b8a8-8a30-49cd-9e74-a278024fdbdb"
-					(reference "SW1")
+					(reference "TARE1")
 					(unit 1)
 				)
@@
 	(symbol
 		(lib_id "Device:R")
-		(at 217.17 73.66 0)
+		(at 223.52 66.04 90)
 		(unit 1)
 		(exclude_from_sim no)
@@
 		(dnp no)
 		(property "Reference" "R6"
-			(at 219.202 73.66 90)
+			(at 223.52 64.008 90)
 			(effects
 				(font
@@
 		)
 		(property "Value" "10k"
-			(at 215.138 73.66 90)
+			(at 223.52 68.072 90)
 			(effects
 				(font
@@
 		)
 		(property "Footprint" "PCM_JLCPCB:R_0603"
-			(at 215.392 73.66 90)
+			(at 223.52 67.818 90)
 			(effects
 				(font
@@
 		)
 		(property "Datasheet" "~"
-			(at 217.17 73.66 0)
+			(at 223.52 66.04 0)
 			(effects
 				(font
@@
 		)
 		(property "Description" "Resistor"
-			(at 217.17 73.66 0)
+			(at 223.52 66.04 0)
 			(effects
 				(font
@@
 			)
 		)
-		(property "Footprint" "Connector_Wire:SolderWire-0.1sqmm_1x02_P3.6mm_D0.4mm_OD1mm"
+		(property "Footprint" "Connector_Molex:Molex_PicoBlade_53048-0210_1x02_P1.25mm_Horizontal"
 			(at 265.43 120.65 0)
 			(effects
@@
 			)
 		)
-		(property "Footprint" "Connector_Wire:SolderWire-0.1sqmm_1x05_P3.6mm_D0.4mm_OD1mm"
+		(property "Footprint" "Connector_PinHeader_2.54mm:PinHeader_1x05_P2.54mm_Vertical"
 			(at 73.66 83.82 0)
 			(effects

Commit message: Breakout xiao pins
Parts:
- added J2: Conn_01x04, Connector_PinHeader_2.54mm:PinHeader_1x04_P2.54mm_Vertical, symbol Connector_Generic:Conn_01x04
Connections:
- net at U2.1 (GPIO2/A0/D0): now also J2.1 (Pin_1)
- net at U2.2 (GPIO3/A1/D1): now also J2.2 (Pin_2)
- net at U2.3 (GPIO4/A2/D2): now also J2.3 (Pin_3)
- net at U2.4 (GPIO5/A3/D3): now also J2.4 (Pin_4)
Other:
- note added: "Generic Breakout"
Changed lines of the file:
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@@
 	(text "IO: 2.7-5.5V"
 		(exclude_from_sim no)
-		(at 260.858 100.33 0)
+		(at 193.04 114.3 0)
 		(effects
 			(font
@@
 		)
 	)
+	(text "Generic\nBreakout"
+		(exclude_from_sim no)
+		(at 275.59 98.806 0)
+		(effects
+			(font
+				(size 1.27 1.27)
+			)
+		)
+	)
 	(text "= 3.08V"
 		(exclude_from_sim no)
@@
 	(text "VCC: 2.7-5.5V"
 		(exclude_from_sim no)
-		(at 260.858 97.79 0)
+		(at 193.04 111.76 0)
 		(effects
 			(font
@@
 	(wire
 		(pts
+			(xy 257.81 97.79) (xy 264.16 97.79)
+		)
+		(stroke
+			(width 0)
+			(type default)
+		)
+	)
+	(wire
+		(pts
 			(xy 101.6 152.4) (xy 101.6 156.21)
 		)
@@
 	(wire
 		(pts
+			(xy 264.16 101.6) (xy 264.16 100.33)
+		)
+		(stroke
+			(width 0)
+			(type default)
+		)
+	)
+	(wire
+		(pts
 			(xy 257.81 82.55) (xy 280.67 82.55)
 		)
@@
 	(wire
 		(pts
+			(xy 264.16 93.98) (xy 264.16 95.25)
+		)
+		(stroke
+			(width 0)
+			(type default)
+		)
+	)
+	(wire
+		(pts
 			(xy 157.48 114.3) (xy 157.48 132.08)
 		)
@@
 	(wire
 		(pts
+			(xy 264.16 105.41) (xy 264.16 102.87)
+		)
+		(stroke
+			(width 0)
+			(type default)
+		)
+	)
+	(wire
+		(pts
 			(xy 127 53.34) (xy 127 50.8)
 		)
@@
 	(wire
 		(pts
+			(xy 257.81 105.41) (xy 264.16 105.41)
+		)
+		(stroke
+			(width 0)
+			(type default)
+		)
+	)
+	(wire
+		(pts
 			(xy 88.9 119.38) (xy 88.9 83.82)
 		)
@@
 	(wire
 		(pts
+			(xy 257.81 93.98) (xy 264.16 93.98)
+		)
+		(stroke
+			(width 0)
+			(type default)
+		)
+	)
+	(wire
+		(pts
 			(xy 187.96 88.9) (xy 193.04 88.9)
 		)
@@
 	(wire
 		(pts
+			(xy 257.81 101.6) (xy 264.16 101.6)
+		)
+		(stroke
+			(width 0)
+			(type default)
+		)
+	)
+	(wire
+		(pts
 			(xy 274.32 86.36) (xy 257.81 86.36)
 		)
@@
 					(unit 1)
 				)
+			)
+		)
+	)
+	(symbol
+		(lib_id "Connector_Generic:Conn_01x04")
+		(at 269.24 100.33 0)
+		(mirror x)
+		(unit 1)
+		(exclude_from_sim no)
+		(in_bom yes)
+		(on_board yes)
+		(dnp no)
+		(property "Reference" "J2"
+			(at 268.224 92.456 0)
+			(effects
+				(font
+					(size 1.27 1.27)
+				)
+				(justify left)
+			)
+		)
+		(property "Value" "Conn_01x04"
+			(at 271.78 97.7901 0)
+			(effects
+				(font
+					(size 1.27 1.27)
+				)
+				(justify left)
+				(hide yes)
+			)
+		)
+		(property "Footprint" "Connector_PinHeader_2.54mm:PinHeader_1x04_P2.54mm_Vertical"
+			(at 268.478 109.474 0)
+			(effects
+				(font
+					(size 1.27 1.27)
+				)
+				(hide yes)
+			)
+		)
+		(property "Datasheet" "~"
+			(at 269.24 100.33 0)
+			(effects
+				(font
+					(size 1.27 1.27)
+				)
+				(hide yes)
+			)
+		)
+		(property "Description" "Generic connector, single row, 01x04, script generated (kicad-library-utils/schlib/autogen/connector/)"
+			(at 269.24 100.33 0)
+			(effects
+				(font
+					(size 1.27 1.27)
+				)
+				(hide yes)
+			)
+		)
+		(pin "3"
+		)
+		(pin "4"
+		)
+		(pin "1"
+		)
+		(pin "2"
+		)
+		(instances
+			(project ""
+				(path "/7828b8a8-8a30-49cd-9e74-a278024fdbdb"
+					(reference "J2")
+					(unit 1)
+				)

Commit message: mito V2 pcb
Parts:
- removed J2: Conn_01x04, Connector_PinHeader_2.54mm:PinHeader_1x04_P2.54mm_Vertical, symbol Connector_Generic:Conn_01x04
- added J2: Conn_01x06, Connector_PinHeader_2.54mm:PinHeader_1x06_P2.54mm_Vertical, symbol Connector_Generic:Conn_01x06
- J1: footprint Connector_Molex:Molex_PicoBlade_53048-0210_1x02_P1.25mm_Horizontal -> Connector_Wire:SolderWire-0.1sqmm_1x02_P3.6mm_D0.4mm_OD1mm_Relief
Connections:
- net GND: now also J2.5 (Pin_5)
- net VCC: now also U1.15 (RATE), J2.6 (Pin_6)
- net at PWR1.2 (A): now also U2.15 (Bat+); no longer J1.1 (Pin_1)
- net at PWR1.3 (B): now also J1.1 (Pin_1); no longer U2.15 (Bat+)
- net at U2.1 (GPIO2/A0/D0): now also J2.1 (Pin_1)
- net at U2.2 (GPIO3/A1/D1): now also J2.2 (Pin_2)
- net at U2.3 (GPIO4/A2/D2): now also J2.3 (Pin_3)
- net at U2.4 (GPIO5/A3/D3): now also J2.4 (Pin_4)
Other:
- note added: "XIAO Breakout"
- note removed: "Generic Breakout"
